File: hw/BBB_CNC.brd (EAGLE design)
At the start: 100 x 100 mm, 46 parts, among them IC1 74HCT125D, IC2 74HCT125D, T1 2N7002K, T2 2N7002K, T3 2N7002K, T4 2N7002K, T5 2N7002K

Commit message: modified v1, finished pcb
Parts:
- moved T4 6.30 mm to (2.10, 13.0)
- moved T5 5.40 mm to (2.10, 17.1)
- moved JP1 2.41 mm to (15.4, 2.90)
- moved R4 1.24 mm to (6.60, 7.90)
- moved JP2 0.20 mm to (4.30, 2.90)
Routing:
- net N$9: track 2.88 -> 9.45 mm, vias 0 -> 1
- net DO_ESTOP_SWITCH: track 114.7 -> 109.5 mm
- net GND: track 0.00 -> 4.32 mm, vias 37 -> 38
- net N$5: track 3.17 -> 5.90 mm, vias 0 -> 1
- net +5V: track 172.6 -> 174.7 mm
- net DI_ESTOP: track 106.2 -> 104.1 mm
- net N$8: track 7.48 -> 5.58 mm
- net I_MACHINE_POWER1: track 40.5 -> 41.6 mm, vias 2 -> 3
- net DO_X_STEP_BUFF: vias 2 -> 1
Other:
- board text added: "Z-Max/Min"
- board text removed: "Z-Min/Max"

Commit message: V2, gerber files for Itead
Parts:
- removed SP1: SP4, SchlegelAr_Master:SP4
- moved JP3 1.20 mm to (21.6, 92.2)
- moved JP4 1.20 mm to (33.6, 92.2)
- moved R11 1.20 mm to (19.0, 84.1)
- moved R12 1.20 mm to (24.6, 84.2)
- moved R14 1.20 mm to (31.9, 84.1)
- moved R15 1.20 mm to (37.2, 84.0)
- moved LED4 0.40 mm to (24.5, 8.80)
- moved R7 0.30 mm to (27.2, 7.30)
Connections:
- removed net DO_!X_EN_BUFF: SP1.P$4, X5.1
- removed net DO_!Y_EN_BUFF: SP1.P$2, X5.3
- removed net DO_!Z_EN_BUFF: SP1.P$3, X5.5
- removed net N$18: IC2.3, R9.1, SP1.P$1
- new net DO_!AXIS_EN_BUFF: IC2.3, R9.1, X5.1, X5.3, X5.5
Routing:
- net DO_!AXIS_EN_BUFF: track 0.00 -> 72.1 mm
- net DO_!Z_EN_BUFF: track 27.6 -> 0.00 mm, vias 1 -> 0
- net N$18: track 25.5 -> 0.00 mm
- net DO_!Y_EN_BUFF: track 17.6 -> 0.00 mm, vias 1 -> 0
- net DO_!X_EN_BUFF: track 8.33 -> 0.00 mm, vias 1 -> 0
- net +5V: track 174.7 -> 166.8 mm
- net +3V3: track 297.2 -> 292.7 mm
- net DO_MACHINE_POWER: track 55.8 -> 54.4 mm
- net DI_Y_MIN: track 19.3 -> 18.1 mm
- net DI_X_MAX: track 37.6 -> 36.4 mm
- net DI_Y_MAX: track 63.6 -> 62.4 mm
- net DO_X_STEP_BUFF: track 31.1 -> 30.2 mm
- net DI_X_MIN: track 23.6 -> 23.0 mm
- net DI_POWER_BUTTON: track 58.3 -> 57.8 mm, vias 2 -> 1
- net GND: vias 38 -> 43
- removed copper zone on layer 1, net N$11
- removed copper zone on layer 1, net N$13
- removed copper zone on layer 1, net N$14
- removed copper zone on layer 1, net N$15
- removed copper zone on layer 1, net N$16
- removed copper zone on layer 1, net N$17
- removed copper zone on layer 1, net N$19
- removed copper zone on layer 1, net N$20
- removed copper zone on layer 1, net N$21
- removed copper zone on layer 1, net N$22
- removed copper zone on layer 1, net N$23
- removed copper zone on layer 1, net N$24
- removed copper zone on layer 1, net N$4
- removed copper zone on layer 1, net N$6
- removed copper zone on layer 16, net N$7
Other:
- board text added: "+ - AUX-Out"
- board text added: "-+ -+ Z-Max/Min"
- board text added: "BBB_CNC V2 Armin Schlegel 08.07.2014"
- board text added: "DIR_X - +"
- board text added: "DIR_Y - +"
- board text added: "DIR_Z - +"
- board text added: "EN_X - +"
- board text added: "EN_Y - +"
- board text added: "EN_Z - +"
- board text added: "Reset"
- board text added: "ST_X - +"
- board text added: "ST_Y - +"
- board text added: "ST_Z - +"
- board text added: "X-Max/Min -+ -+"
- board text added: "Y-Max/Min -+ -+"
- board text added: "Z-Probe -+"
- board text removed: "+ - AUX"
- board text removed: "BBB_CNC V1 Armin Schlegel 06.07.2014"
- board text removed: "DIR_X"
- board text removed: "DIR_Y"
- board text removed: "DIR_Z"
- board text removed: "EN_X"
- board text removed: "EN_Y"
- board text removed: "EN_Z"
- board text removed: "ST_X"
- board text removed: "ST_Y"
- board text removed: "ST_Z"
- board text removed: "Z-Max/Min"
- board text removed: "ZProbe -+"
