File: hw/BBB_CNC.sch (EAGLE design)
At the start: 46 parts, among them IC1 74HCT125D, IC2 74HCT125D, T1 2N7002K, T2 2N7002K, T3 2N7002K, T4 2N7002K, T5 2N7002K

Commit message: modified v1, finished pcb
Connections:
- net DO_!AXIS_EN: now also IC2A.I; no longer IC2C.I
- net DO_!X_EN_BUFF: now also X5-1.KL; no longer X3-5.KL
- net DO_!Y_EN_BUFF: now also X5-3.KL; no longer X4-5.KL
- net DO_AUX1: no longer X1-1.KL
- net DO_AUX1_BUFF: now also X1-1.KL
- net DO_X_DIR: now also IC1A.I; no longer IC1B.I
- net DO_X_DIR_BUFF: now also IC1A.O, X4-1.KL; no longer IC1B.O, X3-3.KL
- net DO_X_STEP: now also IC1C.I; no longer IC1A.I
- net DO_X_STEP_BUFF: now also IC1C.O; no longer IC1A.O
- net DO_Y_DIR: now also IC1B.I; no longer IC1D.I
- net DO_Y_DIR_BUFF: now also IC1B.O; no longer IC1D.O
- net DO_Y_STEP: now also IC2C.I; no longer IC1C.I
- net DO_Y_STEP_BUFF: now also IC2C.O, X3-3.KL; no longer IC1C.O, X4-1.KL
- net DO_Z_DIR: now also IC1D.I; no longer IC2B.I
- net DO_Z_DIR_BUFF: now also IC1D.O, X4-5.KL; no longer IC2B.O, X5-3.KL
- net DO_Z_STEP: now also IC2B.I; no longer IC2A.I
- net DO_Z_STEP_BUFF: now also IC2B.O, X3-5.KL; no longer IC2A.O, X5-1.KL
- net N$18: now also IC2A.O; no longer IC2C.O
Other:
- moved on the sheet: R9

Commit message: V2, gerber files for Itead
Parts:
- removed SP1: SP4, SchlegelAr_Master:SP4
Connections:
- removed net DO_!X_EN_BUFF: SP1.4, X5-1.KL
- removed net DO_!Y_EN_BUFF: SP1.2, X5-3.KL
- removed net DO_!Z_EN_BUFF: SP1.3, X5-5.KL
- removed net N$18: IC2A.O, R9.1, SP1.1
- new net DO_!AXIS_EN_BUFF: IC2A.O, R9.1, X5-1.KL, X5-3.KL, X5-5.KL
Other:
- note added: "Armin Schlegel 08.07.2014"
- note added: "Beaglebone Black V2 CNC Cape Derived from CRAMPS V2.1"
- note removed: "Armin Schlegel 04.07.2014"
- note removed: "Beaglebone Black V1 CNC Cape Derived from CRAMPS V2.1"
Changed lines of the file:
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@@
 <part name="P+3" library="supply1" deviceset="+5V" device=""/>
 <part name="GND7" library="supply1" deviceset="GND" device=""/>
-<part name="SP1" library="SchlegelAr_Master" deviceset="SP4" device=""/>
 <part name="FRAME3" library="frames" deviceset="A4L-LOC" device=""/>
 <part name="T2" library="zetex" deviceset="NMOSSOT23" device="" value="2N7002K"/>
@@
 <text x="180.34" y="93.98" size="1.778" layer="97">Status LED</text>
 <text x="205.74" y="93.98" size="1.778" layer="97">Power LED</text>
-<text x="162.56" y="12.7" size="2.54" layer="97">Beaglebone Black V1
+<text x="66.04" y="167.64" size="3.81" layer="97">Beaglebone Black</text>
+<text x="162.56" y="12.7" size="2.54" layer="97">Beaglebone Black V2
 CNC Cape
 Derived from CRAMPS V2.1</text>
-<text x="66.04" y="167.64" size="3.81" layer="97">Beaglebone Black</text>
 <text x="167.64" y="5.08" size="2.54" layer="97">Armin Schlegel
-04.07.2014</text>
+08.07.2014</text>
 </plain>
 <instances>
@@
 <text x="142.24" y="144.78" size="2.54" layer="97">Machine Power
 Status LED</text>
-<text x="162.56" y="12.7" size="2.54" layer="97">Beaglebone Black V1
+<text x="162.56" y="12.7" size="2.54" layer="97">Beaglebone Black V2
 CNC Cape
 Derived from CRAMPS V2.1</text>
 <text x="167.64" y="5.08" size="2.54" layer="97">Armin Schlegel
-04.07.2014</text>
+08.07.2014</text>
 </plain>
 <instances>
@@
 <text x="50.8" y="30.48" size="2.54" layer="97">74HCT125 has 25mA per output
 That is enough for optocouplers on the TB6560 Board </text>
-<text x="162.56" y="12.7" size="2.54" layer="97">Beaglebone Black V1
+<text x="162.56" y="12.7" size="2.54" layer="97">Beaglebone Black V2
 CNC Cape
 Derived from CRAMPS V2.1</text>
 <text x="167.64" y="5.08" size="2.54" layer="97">Armin Schlegel
-04.07.2014</text>
+08.07.2014</text>
 </plain>
 <instances>
@@
 <instance part="P+3" gate="1" x="134.62" y="73.66"/>
 <instance part="GND7" gate="1" x="134.62" y="43.18"/>
-<instance part="SP1" gate="G$1" x="160.02" y="154.94"/>
 <instance part="R9" gate="G$1" x="152.4" y="162.56" rot="R90"/>
 <instance part="P+4" gate="1" x="152.4" y="172.72"/>
@@
 </segment>
 </net>
-<net name="N$18" class="0">
-<segment>
-<pinref part="SP1" gate="G$1" pin="1"/>
+<net name="DO_!AXIS_EN_BUFF" class="0">
+<segment>
 <pinref part="R9" gate="G$1" pin="1"/>
 <wire x1="147.32" y1="154.94" x2="152.4" y2="154.94" width="0.1524" layer="91"/>
@@
 <junction x="152.4" y="154.94"/>
 <pinref part="IC2" gate="A" pin="O"/>
+<label x="157.48" y="154.94" size="1.27" layer="95" xref="yes"/>
 </segment>
 </net>
@@
 <wire x1="45.72" y1="132.08" x2="40.64" y2="132.08" width="0.1524" layer="91"/>
 <pinref part="IC1" gate="B" pin="I"/>
-</segment>
-</net>
-<net name="DO_!X_EN_BUFF" class="0">
-<segment>
-<pinref part="SP1" gate="G$1" pin="4"/>
-<wire x1="160.02" y1="157.48" x2="160.02" y2="160.02" width="0.1524" layer="91"/>
-<wire x1="160.02" y1="160.02" x2="165.1" y2="160.02" width="0.1524" layer="91"/>
-<label x="165.1" y="160.02" size="1.27" layer="95" xref="yes"/>
-</segment>
-</net>
-<net name="DO_!Y_EN_BUFF" class="0">
-<segment>
-<pinref part="SP1" gate="G$1" pin="2"/>
-<wire x1="162.56" y1="154.94" x2="165.1" y2="154.94" width="0.1524" layer="91"/>
-<label x="165.1" y="154.94" size="1.27" layer="95" xref="yes"/>
-</segment>
-</net>
-<net name="DO_!Z_EN_BUFF" class="0">
-<segment>
-<pinref part="SP1" gate="G$1" pin="3"/>
-<wire x1="160.02" y1="152.4" x2="160.02" y2="149.86" width="0.1524" layer="91"/>
-<wire x1="160.02" y1="149.86" x2="165.1" y2="149.86" width="0.1524" layer="91"/>
-<label x="165.1" y="149.86" size="1.27" layer="95" xref="yes"/>
 </segment>
 </net>
@@
 <text x="53.34" y="33.02" size="2.54" layer="97">Auxillary Output
 e.g. Spindle Control</text>
-<text x="162.56" y="12.7" size="2.54" layer="97">Beaglebone Black V1
+<text x="162.56" y="12.7" size="2.54" layer="97">Beaglebone Black V2
 CNC Cape
 Derived from CRAMPS V2.1</text>
@@
 that are normally closed</text>
 <text x="167.64" y="5.08" size="2.54" layer="97">Armin Schlegel
-04.07.2014</text>
+08.07.2014</text>
 </plain>
 <instances>
@@
 </segment>
 </net>
-<net name="DO_!X_EN_BUFF" class="0">
-<segment>
-<label x="27.94" y="73.66" size="1.27" layer="95" rot="R180" xref="yes"/>
-<wire x1="35.56" y1="73.66" x2="27.94" y2="73.66" width="0.1524" layer="91"/>
-<pinref part="X5" gate="-1" pin="KL"/>
-</segment>
-</net>
 <net name="DO_Y_STEP_BUFF" class="0">
 <segment>
@@
 </segment>
 </net>
-<net name="DO_!Y_EN_BUFF" class="0">
-<segment>
-<label x="27.94" y="68.58" size="1.27" layer="95" rot="R180" xref="yes"/>
-<wire x1="35.56" y1="68.58" x2="27.94" y2="68.58" width="0.1524" layer="91"/>
-<pinref part="X5" gate="-3" pin="KL"/>
-</segment>
-</net>
 <net name="DO_Z_STEP_BUFF" class="0">
 <segment>
@@
 <wire x1="35.56" y1="104.14" x2="27.94" y2="104.14" width="0.1524" layer="91"/>
 <pinref part="X4" gate="-5" pin="KL"/>
-</segment>
-</net>
-<net name="DO_!Z_EN_BUFF" class="0">
-<segment>
-<pinref part="X5" gate="-5" pin="KL"/>
-<wire x1="35.56" y1="63.5" x2="27.94" y2="63.5" width="0.1524" layer="91"/>
-<label x="27.94" y="63.5" size="1.27" layer="95" rot="R180" xref="yes"/>
 </segment>
 </net>
@@
 </segment>
 </net>
+<net name="DO_!AXIS_EN_BUFF" class="0">
+<segment>
+<pinref part="X5" gate="-1" pin="KL"/>
+<wire x1="35.56" y1="73.66" x2="27.94" y2="73.66" width="0.1524" layer="91"/>
+<label x="27.94" y="73.66" size="1.27" layer="95" rot="R180" xref="yes"/>
+</segment>
+<segment>
+<pinref part="X5" gate="-3" pin="KL"/>
+<wire x1="35.56" y1="68.58" x2="27.94" y2="68.58" width="0.1524" layer="91"/>
+<label x="27.94" y="68.58" size="1.27" layer="95" rot="R180" xref="yes"/>
+</segment>
+<segment>
+<pinref part="X5" gate="-5" pin="KL"/>
+<wire x1="35.56" y1="63.5" x2="27.94" y2="63.5" width="0.1524" layer="91"/>
+<label x="27.94" y="63.5" size="1.27" layer="95" rot="R180" xref="yes"/>
+</segment>
+</net>
