File: hw/BBB_CNC_V3.brd (EAGLE design)
At the start: 100 x 100 mm, 45 parts, among them IC1 74HCT125D, IC2 74HCT125D, T1 2N7002K, T2 2N7002K, T3 2N7002K, T4 2N7002K, T5 2N7002K

Commit message: updated gerber files to V3
Parts:
- added JP9: (no value), pinhead:1X02
- moved R4 0.73 mm to (6.80, 8.60)
Connections:
- net +5V: now also JP9.1
- net GND: now also JP9.2
Routing:
- net +5V: track 166.8 -> 171.2 mm
- net I_MACHINE_POWER1: track 41.6 -> 42.5 mm
- net DI_ESTOP: track 104.1 -> 103.5 mm
Other:
- board text added: "5V + -"
- board text added: "ESTOP"
- board text added: "Machine PWR"
Changed lines of the file:
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@@
 <text x="36.2" y="38" size="1.778" layer="21" ratio="15">Z-Probe
 -+ </text>
-<text x="35.2" y="2.7" size="1.778" layer="21" ratio="15"> -+ -+
+<text x="36.5" y="2.8" size="1.778" layer="21" ratio="15">-+ -+
 Z-Max/Min</text>
 <text x="89.5" y="29" size="1.778" layer="21" ratio="15" rot="R90">EN_X
@@
 <text x="14.2" y="99.2" size="1.778" layer="21" ratio="15" align="top-left">X-Max/Min
   -+ -+</text>
+<text x="13" y="26.3" size="1.778" layer="21" ratio="15">5V
++ -</text>
+<text x="0.5" y="4.8" size="1.778" layer="21" ratio="15">ESTOP</text>
+<text x="18.7" y="0.9" size="1.778" layer="21" ratio="15">Machine PWR</text>
 </plain>
 <attributes>
@@
 <attribute name="VALUE" x="5.665" y="10.295" size="1.27" layer="27"/>
 </element>
-<element name="R4" library="rcl" package="R0603" value="10k" x="6.6" y="7.9" rot="R180"/>
+<element name="R4" library="rcl" package="R0603" value="10k" x="6.8" y="8.6" rot="R180"/>
 <element name="LED3" library="led" package="SML0805" value="GREEN" x="30.6" y="8.8" smashed="yes">
 <attribute name="NAME" x="30.5" y="10.3" size="1.27" layer="25" rot="R90"/>
@@
 <attribute name="VALUE" x="38.965" y="28.495" size="1.27" layer="27"/>
 </element>
+<element name="JP9" library="pinhead" package="1X02" value="" x="15.3" y="24.2"/>
 </elements>
 <signals>
@@
 <via x="13.2384" y="16.4656" extent="1-16" drill="0.6" diameter="1.016" shape="octagon"/>
 <contactref element="IC2" pad="10"/>
+<contactref element="JP9" pad="2"/>
 </signal>
 <signal name="DI_X_MAX">
@@
 <wire x1="56.1" y1="40.2" x2="36.6" y2="40.2" width="0.6096" layer="1"/>
 <wire x1="36.6" y1="40.2" x2="33.7" y2="37.3" width="0.6096" layer="1"/>
-<wire x1="31" y1="20.3" x2="11.8" y2="20.3" width="0.6096" layer="1"/>
+<wire x1="31" y1="20.3" x2="12.9" y2="20.3" width="0.6096" layer="1"/>
+<wire x1="12.9" y1="20.3" x2="11.8" y2="20.3" width="0.6096" layer="1"/>
 <wire x1="11.8" y1="20.3" x2="8.7" y2="17.2" width="0.6096" layer="1"/>
 <wire x1="78.3" y1="84.6" x2="79.9" y2="83" width="0.8128" layer="16"/>
@@
 <wire x1="79.9" y1="79.5" x2="81.9" y2="77.5" width="0.8128" layer="16"/>
 <wire x1="81.9" y1="77.5" x2="83.4" y2="77.5" width="0.8128" layer="16"/>
+<contactref element="JP9" pad="1"/>
+<wire x1="14.03" y1="24.2" x2="14.03" y2="21.43" width="0.6096" layer="1"/>
+<wire x1="14.03" y1="21.43" x2="12.9" y2="20.3" width="0.6096" layer="1"/>
 </signal>
 <signal name="N$1">
@@
 <wire x1="46.6" y1="61.1" x2="46.6" y2="72.325" width="0.8128" layer="1"/>
 <wire x1="46.6" y1="72.325" x2="46.37" y2="72.555" width="0.8128" layer="1"/>
-<wire x1="5.45" y1="9.05" x2="4.9" y2="9.6" width="0.65" layer="1"/>
 <wire x1="4.9" y1="9.6" x2="4.5" y2="9.6" width="0.65" layer="1"/>
 <wire x1="4.5" y1="9.6" x2="4.4" y2="9.7" width="0.65" layer="1"/>
 <wire x1="4.4" y1="10.4" x2="4.4" y2="9.7" width="0.8128" layer="16"/>
-<wire x1="5.75" y1="7.9" x2="5.75" y2="8.75" width="0.6096" layer="1"/>
-<wire x1="5.75" y1="8.75" x2="5.45" y2="9.05" width="0.6096" layer="1"/>
 <wire x1="4.4" y1="10.4" x2="4.4" y2="16.2" width="0.6096" layer="16"/>
 <wire x1="4.4" y1="16.2" x2="5.5" y2="17.3" width="0.6096" layer="16"/>
+<wire x1="5.95" y1="8.6" x2="5.9" y2="8.6" width="0.6096" layer="1"/>
+<wire x1="5.9" y1="8.6" x2="4.9" y2="9.6" width="0.6096" layer="1"/>
 </signal>
 <signal name="DO_X_STEP">
@@
 <wire x1="9.2" y1="11.6" x2="9.2" y2="7.8762" width="0.65" layer="1"/>
 <wire x1="9.2" y1="7.8762" x2="9.3602" y2="7.716" width="0.65" layer="1"/>
-<wire x1="7.45" y1="7.9" x2="9.1762" y2="7.9" width="0.6096" layer="1"/>
 <wire x1="9.1762" y1="7.9" x2="9.3602" y2="7.716" width="0.6096" layer="1"/>
-<wire x1="7.45" y1="7.9" x2="7.45" y2="6.65" width="0.6096" layer="1"/>
 <wire x1="7.45" y1="6.65" x2="6.6" y2="5.8" width="0.6096" layer="1"/>
 <via x="6.6" y="5.8" extent="1-16" drill="0.6" diameter="1.016" shape="octagon"/>
@@
 <wire x1="10.1" y1="10.6" x2="15" y2="10.6" width="0.8128" layer="16"/>
 <wire x1="15" y1="10.6" x2="16.3" y2="11.9" width="0.8128" layer="16"/>
+<wire x1="9.1762" y1="7.9" x2="8.35" y2="7.9" width="0.6096" layer="1"/>
+<wire x1="8.35" y1="7.9" x2="7.65" y2="8.6" width="0.6096" layer="1"/>
+<wire x1="7.45" y1="6.65" x2="7.45" y2="8.4" width="0.6096" layer="1"/>
+<wire x1="7.45" y1="8.4" x2="7.65" y2="8.6" width="0.6096" layer="1"/>
 </signal>
 <signal name="DO_X_STEP_BUFF">
