File: hw/BBB_CNC_V3.sch (EAGLE design)
At the start: 45 parts, among them IC1 74HCT125D, IC2 74HCT125D, T1 2N7002K, T2 2N7002K, T3 2N7002K, T4 2N7002K, T5 2N7002K

Commit message: updated gerber files to V3
Parts:
- added JP9: (no value), pinhead:PINHD-1X2
Connections:
- net +5V: now also JP9.1
- net GND: now also JP9.2
Changed lines of the file:
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@@
 <part name="R13" library="rcl" deviceset="R-EU_" device="R0603" value="4k7"/>
 <part name="+3V9" library="supply1" deviceset="+3V3" device=""/>
+<part name="JP9" library="pinhead" deviceset="PINHD-1X2" device=""/>
+<part name="GND12" library="supply1" deviceset="GND" device=""/>
+<part name="P+7" library="supply1" deviceset="+5V" device=""/>
 </parts>
 <sheets>
@@
 <instance part="P+5" gate="1" x="127" y="165.1"/>
 <instance part="P+6" gate="1" x="137.16" y="165.1"/>
+<instance part="JP9" gate="G$1" x="43.18" y="147.32" rot="MR0"/>
+<instance part="GND12" gate="1" x="53.34" y="142.24"/>
+<instance part="P+7" gate="1" x="53.34" y="160.02"/>
 </instances>
 <busses>
@@
 <pinref part="GND10" gate="1" pin="GND"/>
 <wire x1="93.98" y1="55.88" x2="93.98" y2="40.64" width="0.1524" layer="91"/>
+</segment>
+<segment>
+<pinref part="JP9" gate="G$1" pin="2"/>
+<pinref part="GND12" gate="1" pin="GND"/>
+<wire x1="45.72" y1="147.32" x2="53.34" y2="147.32" width="0.1524" layer="91"/>
+<wire x1="53.34" y1="147.32" x2="53.34" y2="144.78" width="0.1524" layer="91"/>
 </segment>
 </net>
@@
 <pinref part="P+6" gate="1" pin="+5V"/>
 </segment>
-</net>
+<segment>
+<pinref part="JP9" gate="G$1" pin="1"/>
+<pinref part="P+7" gate="1" pin="+5V"/>
+<wire x1="45.72" y1="149.86" x2="53.34" y2="149.86" width="0.1524" layer="91"/>
+<wire x1="53.34" y1="149.86" x2="53.34" y2="157.48" width="0.1524" layer="91"/>
+</segment>
+</net>
